File: proto-h750.kicad_pcb (KiCad board)
At the start: 2 copper layers, 158 parts, among them J1 Conn_02x08_Odd_Even, J10 Conn_02x02_Odd_Even, J11 Conn_02x02_Odd_Even, J12 Conn_01x02, J13 Conn_01x02, J2 USB_B_Micro, J3 Conn_02x02_Odd_Even, J4 Conn_02x14_Odd_Even, J5 Conn_02x08_Odd_Even, J6 AudioJack3, J7 Conn_02x02_Odd_Even, J8 Screw_Terminal_01x02, J9 AudioJack3, Q1 BS170, Q2 BS170, Q3 BS170, Q4 IRF540N, Q5 BSS138, Q6 MMBT2222, SW1 SW_DIP_x01, SW2 SW_DIP_x01, SW3 SW_DIP_x01, T1 Transformer_1P_1S, U1 STA516BETR, U10 BGA2869, U11 BGA2869, U2 STM32H750VBT6, U3 AP1117-33, U4 LM7805_TO220, U5 LM7812_TO220, U6 LM5134AMF_NOPB, U9 SA612, X1 ASV-xxxMHz, Y1 16MHz, Y2 ECS-10.7-7.5B

Commit message: Almost routed
Parts:
- moved C32 42.4 mm to (126.5, 100.3)
- moved R5 21.2 mm to (123.7, 117.1)
- moved C47 0.25 mm to (117.9, 106.9)
Routing:
- net VCC: track 37.1 -> 210.6 mm, vias 0 -> 4
- net GND: track 880.3 -> 960.5 mm, vias 89 -> 93
- net +24V: track 44.3 -> 103.7 mm, vias 0 -> 2
- net TXV: track 29.3 -> 86.3 mm, vias 0 -> 6
- net A_PWM: track 9.30 -> 54.7 mm, vias 0 -> 3
- net A_PWRDN: track 11.8 -> 42.1 mm, vias 0 -> 2
- net Net-(C20-Pad1): track 0.00 -> 26.7 mm
- net A_FAULT: track 15.2 -> 40.8 mm, vias 0 -> 1
- net MODUL_OUT: track 10.8 -> 35.7 mm
- net Net-(L2-Pad1): track 15.3 -> 30.5 mm
- net Net-(C37-Pad1): track 0.00 -> 12.5 mm
- net MCO: track 97.4 -> 102.9 mm
- net +5V: track 309.1 -> 314.5 mm
- net Net-(C28-Pad1): track 8.13 -> 10.6 mm
- net Net-(C11-Pad1): track 3.95 -> 5.73 mm
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